File: tcvr.kicad_sch (KiCad schematic)
At the start: 32 parts, among them J1 9V, J2 anterna 50 Ohm, Q1 BC817, Q2 2N7002, Q3 PZT2222A, SW1 SW_DPST_x2, U1 LM386, Y1 3579kHz

Commit message: added bolti megrendelési cimkék
Parts:
- added C14: 47n, symbol Device:C
- added R8: 10, symbol Device:R
- C12: value 47u -> 10u
- C13: value C -> 22u
- C3, C4: value C -> 100p
- D1: value FM14 -> FM14 83-07-39
- L1: value 27u -> 27u 93-04-40
- L3: value 2u2 -> 2u2 93-00-07
- Q1: value BC817 -> BC817 86-05-47
- Q3: value PZT2222A -> PZT2222A 86-02-43
- U1: value LM386 -> LM386 89-24-08
- Y1: value 3579kHz -> 3579kHz 40-00-62
Connections:
- net GND: now also R8.2
- net at U1.5: now also C14.2
- new net: C14.1, R8.1
Other:
- moved on the sheet: C5, Q2, R3, R4, Y1
